File: hardware/eda/FlightSimController.kicad_pcb (KiCad board)
At the start: 6 copper layers, 72 x 72 mm, 190 parts, among them J1 Conn_02x14_Odd_Even, J10 RS485 OUT, J2 RP2040 PGM, J3 HDMI_A, J4 Conn_01x40_Shielded, J5 Conn_02x05_Odd_Even, J6 USB_A, J7 RS485 IN, J8 12V_SW, M1 ComputeModule4-CM4, SW1 SW_Push, SW2 SW_Push, U1 MAX485E, U10 TC78H611FNG, U11 TC78H611FNG, U12 MCP3424, U13 TPD2E009, U14 TPD2E009, U15 HDMIULC6-4SC6, U16 HDMIULC6-4SC6, U17 TPD2E009, U18 HDMIULC6-4SC6, U2 TS19371CX6RFG, U3 TSC2007IPWR, U4 LD2980, U5 ADP2303ARDZ-3.3, U6 ADP2303ARDZ-5.0, U7 VN5E160STR-E, U8 IS25LP128F-JBLE, U9 RP2040, Y1 Crystal_GND24_Small

Commit message: Silkscreen Adjustments
Parts:
- added REF**: ESD-Logo_13.2x12mm_SilkScreen, Symbol:ESD-Logo_13.2x12mm_SilkScreen, B.Cu at (142.5, 94.5)
- added REF**: OSHW-Logo2_14.6x12mm_SilkScreen, Symbol:OSHW-Logo2_14.6x12mm_SilkScreen, B.Cu at (167.6, 95.5)
Other:
- board text added: "Copyright Peter Heinrich 2022. This source describes Open Hardware and is licensed under the CERN-OHL-P v2 You may redistribute and modify this documentation and make products using it under the terms of the CERN-OHL-P v2 (https:/cern.ch/cern-ohl). This documentation is distributed WITHOUT ANY EXPRESS OR IMPLIED WARRANTY, INCLUDING OF MERCHANTABILITY, SATISFACTORY QUALITY AND FITNESS FOR A PARTIC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"
- board text added: "FlightSimController Copytight © 2022 by Peter Heinrich Rev A"
- board text added: "STOP! This is an experimental and untested hardware design! At the current state this document is only educational and NOT intended for physical construction of the electronic module. If you nontheless intend to build this early prototype, you do this fully at your own risk."
- board text removed: "FlightSimMod V1.0 Copytight © 2022 by Peter Heinrich"
