File: hardware/eda/CM4_Header.kicad_sch (KiCad schematic)
At the start: 25 parts, among them M1 ComputeModule4-CM4, U15 HDMIULC6-4SC6, U16 HDMIULC6-4SC6, U2 TS19371CX6RFG, U3 TSC2007IPWR

Commit message: Updating Backlight Controller Sense Resistor
Parts:
- M1: MPN DF40C-100DS-0.4V(51) -> DF40C-100DP-0.4V(51); ON_FARNELL 2427679 -> 2427678
- R8: value R -> 4R7; MPN (none) -> CR1206AF/-4R70EAS; ON_FARNELL (none) -> 3223654
Other:
- note added: "Table for R8 ------------ 4R7 -> 20.2 mA (Display 3.5": MCT035G12W320240LML)"
- moved on the sheet: C5, C6, D1, FB2, L1, R7, R8, U2
