File: hardware/eda/GPIO.kicad_sch (KiCad schematic)
At the start: 70 parts, among them U10 TC78H611FNG, U11 TC78H611FNG, U12 MCP3424, U18 HDMIULC6-4SC6

Commit message: Adding Procurement Ordering Information
Parts:
- R50, R51: MPN RC0603FR-074K7L. -> RC0603FR-074K7P; ON_FARNELL 2421876 -> 3951355
Changed lines of the file:
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@@
       (effects (font (size 1.27 1.27)) hide)
     )
-    (property "MPN" "RC0603FR-074K7L." (id 4) (at 261.62 118.11 0)
-      (effects (font (size 1.27 1.27)) hide)
-    )
-    (property "ON_FARNELL" "2421876" (id 5) (at 261.62 118.11 0)
+    (property "MPN" "RC0603FR-074K7P" (id 4) (at 261.62 118.11 0)
+      (effects (font (size 1.27 1.27)) hide)
+    )
+    (property "ON_FARNELL" "3951355" (id 5) (at 261.62 118.11 0)
       (effects (font (size 1.27 1.27)) hide)
     )
@@
       (effects (font (size 1.27 1.27)) hide)
     )
-    (property "MPN" "RC0603FR-074K7L." (id 4) (at 266.7 118.11 0)
-      (effects (font (size 1.27 1.27)) hide)
-    )
-    (property "ON_FARNELL" "2421876" (id 5) (at 266.7 118.11 0)
-      (effects (font (size 1.27 1.27)) hide)
-    )
+    (property "MPN" "RC0603FR-074K7P" (id 4) (at 266.7 118.11 0)
+      (effects (font (size 1.27 1.27)) hide)
+    )
+    (property "ON_FARNELL" "3951355" (id 5) (at 266.7 118.11 0)
+      (effects (font (size 1.27 1.27)) hide)
+    )
