File: hardware/eda/RP2040.kicad_sch (KiCad schematic)
At the start: 25 parts, among them SW1 SW_Push, SW2 SW_Push, U8 IS25LP128F-JBLE, U9 RP2040, Y1 Crystal_GND24_Small

Commit message: Adding Procurement Ordering Information
Parts:
- R67, R68: MPN RC0603FR-074K7L. -> RC0603FR-074K7P; ON_FARNELL 2421876 -> 3951355
Changed lines of the file:
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@@
       (effects (font (size 1.27 1.27)) hide)
     )
-    (property "MPN" "RC0603FR-074K7L." (id 4) (at 193.04 46.99 0)
-      (effects (font (size 1.27 1.27)) hide)
-    )
-    (property "ON_FARNELL" "2421876" (id 5) (at 193.04 46.99 0)
+    (property "MPN" "RC0603FR-074K7P" (id 4) (at 193.04 46.99 0)
+      (effects (font (size 1.27 1.27)) hide)
+    )
+    (property "ON_FARNELL" "3951355" (id 5) (at 193.04 46.99 0)
       (effects (font (size 1.27 1.27)) hide)
     )
@@
       (effects (font (size 1.27 1.27)) hide)
     )
-    (property "MPN" "RC0603FR-074K7L." (id 4) (at 187.96 46.99 0)
-      (effects (font (size 1.27 1.27)) hide)
-    )
-    (property "ON_FARNELL" "2421876" (id 5) (at 187.96 46.99 0)
-      (effects (font (size 1.27 1.27)) hide)
-    )
+    (property "MPN" "RC0603FR-074K7P" (id 4) (at 187.96 46.99 0)
+      (effects (font (size 1.27 1.27)) hide)
+    )
+    (property "ON_FARNELL" "3951355" (id 5) (at 187.96 46.99 0)
+      (effects (font (size 1.27 1.27)) hide)
+    )
